File: eagle/8x8matrix.brd (EAGLE design)
At the start: 60.4 x 60.5 mm, 18 parts

Commit message: update eagle schematic
Parts:
- JP2: value M09 -> (none)
- renumbered U$14 to U1, U$28 to U3, U$29 to U4, U$30 to U5, U$31 to U6, U$9 to U2
Routing:
- net GND: track 157.8 -> 156.5 mm
