File: eagle/8x8matrix.sch (EAGLE design)
At the start: 18 parts

Commit message: update eagle schematic
Parts:
- JP2: value M09 -> (none)
- renumbered U$14 to U1, U$28 to U3, U$29 to U4, U$30 to U5, U$31 to U6, U$9 to U2
Other:
- moved on the sheet: JP2, R1, R2
